File: HARDWARE/ETH1CREF1B/Control.kicad_sch (KiCad schematic)
At the start: 20 parts, among them J301 Conn_02x04_Odd_Even, U303 24LC08

Commit message: Hardware
Parts:
- removed C311, C312, C313: 100n, Capacitor_SMD:C_0603_1608Metric_Pad1.08x0.95mm_HandSolder, symbol Device:C
- removed U? (x3): MCZ33996, symbol ETH1CREF1A:MCZ33996
- removed U?: PCA9557PW, symbol ETH1CREF1A:PCA9557PW
- added J301: Conn_02x04_Odd_Even, Connector_PinHeader_2.54mm:PinHeader_2x04_P2.54mm_Vertical, symbol Connector_Generic:Conn_02x04_Odd_Even
- added U301, U302, U304, U305: MCZ33996, ETH1CREF1B:HSOP-32-1EP_7.5x11.0mm_P0.65mm_ThermalVias, symbol ETH1CREF1B:MCZ33996
- added U306: PCA9557PW, Package_SO:TSSOP-16_4.4x5mm_P0.65mm, symbol ETH1CREF1B:PCA9557PW
- R301: renamed from R?; footprint (none) -> Resistor_SMD:R_0603_1608Metric_Pad0.98x0.95mm_HandSolder
- U303: footprint (none) -> Package_SO:MSOP-8_3x3mm_P0.65mm
- renumbered J301 to J302
Connections:
- net +3.3V: now also C310.1, J301.4 (Pin_4), U301.27 (~{RST}), U301.3 (SOPWR), U302.27 (~{RST}), U302.3 (SOPWR), U304.27 (~{RST}), U304.3 (SOPWR), U305.27 (~{RST}), U305.3 (SOPWR), U306.16 (VDD)
- net +5V: now also J301.2 (Pin_2), U301.6 (VPWR), U302.6 (VPWR), U304.6 (VPWR), U305.6 (VPWR); no longer C310.1
- net GND: now also J301.5 (Pin_5), J301.6 (Pin_6), J301.7 (Pin_7), J301.8 (Pin_8), U301.10 (GND), U301.23 (GND), U301.24 (GND), U301.25 (GND), U301.26 (GND), U301.33 (EP), U301.7 (GND), U301.8 (GND), U301.9 (GND), U302.10 (GND), U302.23 (GND), U302.24 (GND), U302.25 (GND), U302.26 (GND), U302.33 (EP), U302.7 (GND), U302.8 (GND), U302.9 (GND), U304.10 (GND), U304.23 (GND), U304.24 (GND), U304.25 (GND), U304.26 (GND), U304.33 (EP), U304.7 (GND), U304.8 (GND), U304.9 (GND), U305.10 (GND), U305.23 (GND), U305.24 (GND), U305.25 (GND), U305.26 (GND), U305.33 (EP), U305.7 (GND), U305.8 (GND), U305.9 (GND), U306.3 (A0), U306.4 (A1), U306.5 (A2), U306.8 (VSS)
- net I2C_SCL: now also U306.1 (SCL)
- net I2C_SDA: now also U306.2 (SDA)
- net at R301.2: now also U306.15 (~{RESET})
- net SPI_SCK: now reaches J302.2 (Pin_2)
- net SPI_SCK: now also U301.11 (SCLK), U302.11 (SCLK), U304.11 (SCLK), U305.11 (SCLK)
- net SPI_MISO: now reaches J302.4 (Pin_4)
- net SPI_MISO: now also U301.22 (SO), U302.22 (SO), U304.22 (SO), U305.22 (SO)
- net SPI_MOSI: now reaches J302.6 (Pin_6)
- net SPI_MOSI: now also U301.19 (SI), U302.19 (SI), U304.19 (SI), U305.19 (SI)
- net I2C_WP renamed EEPROM_WP
- net EEPROM_WP: now also U306.11 (IO4)
- new net OUT0: U304.1 (OUT0)
- new net OUT1: U304.2 (OUT1)
- new net OUT10: U304.20 (OUT10)
- new net OUT11: U304.21 (OUT11)
- new net OUT12: U304.28 (OUT12)
- new net OUT13: U304.29 (OUT13)
- new net OUT14: U304.31 (OUT14)
- new net OUT15: U304.32 (OUT15)
- new net OUT16: U305.1 (OUT0)
- new net OUT17: U305.2 (OUT1)
- new net OUT18: U305.4 (OUT2)
- new net OUT19: U305.5 (OUT3)
- new net OUT2: U304.4 (OUT2)
- new net OUT20: U305.12 (OUT4)
- new net OUT21: U305.13 (OUT5)
- new net OUT22: U305.15 (OUT6)
- new net OUT23: U305.16 (OUT7)
- new net OUT3: U304.5 (OUT3)
- new net OUT4: U304.12 (OUT4)
- new net OUT5: U304.13 (OUT5)
- new net OUT6: U304.15 (OUT6)
- new net OUT7: U304.16 (OUT7)
- new net OUT8: U304.17 (OUT8)
- new net OUT9: U304.18 (OUT9)
- new net RSET0: U301.1 (OUT0)
- new net RSET1: U301.2 (OUT1)
- new net RSET10: U301.20 (OUT10)
- new net RSET11: U301.21 (OUT11)
- new net RSET12: U301.28 (OUT12)
- new net RSET13: U301.29 (OUT13)
- new net RSET14: U301.31 (OUT14)
- new net RSET15: U301.32 (OUT15)
- new net RSET16: U302.1 (OUT0)
- new net RSET17: U302.2 (OUT1)
- new net RSET18: U302.4 (OUT2)
- new net RSET19: U302.5 (OUT3)
- new net RSET2: U301.4 (OUT2)
- new net RSET20: U302.12 (OUT4)
- new net RSET21: U302.13 (OUT5)
- new net RSET22: U302.15 (OUT6)
- new net RSET23: U302.16 (OUT7)
- new net RSET24: U302.17 (OUT8)
- new net RSET25: U302.18 (OUT9)
- new net RSET26: U302.20 (OUT10)
- new net RSET27: U302.21 (OUT11)
- new net RSET28: U302.28 (OUT12)
- new net RSET29: U302.29 (OUT13)
- new net RSET3: U301.5 (OUT3)
- new net RSET4: U301.12 (OUT4)
- new net RSET5: U301.13 (OUT5)
- new net RSET6: U301.15 (OUT6)
- new net RSET7: U301.16 (OUT7)
- new net RSET8: U301.17 (OUT8)
- new net RSET9: U301.18 (OUT9)
- new net SPI_CS0: U301.14 (~{CS}), U306.6 (IO0)
- new net SPI_CS1: U302.14 (~{CS}), U306.7 (IO1)
- new net SPI_CS2: U304.14 (~{CS}), U306.9 (IO2)
- new net SPI_CS3: U305.14 (~{CS}), U306.10 (IO3)
- no-connect marks 3 -> 19
Other:
- moved on the sheet: J302
