File: HARDWARE/ETH1CREF1B/ETH1CREF1B.kicad_sch (KiCad schematic)
At the start: 0 parts

Commit message: Hardware
Parts:
- added H101, H102, H103: MountingHole, MountingHole:MountingHole_3.2mm_M3_DIN965_Pad_TopBottom, symbol Mechanical:MountingHole
Other:
- sheet Control ports: added OUT[0..23], RSET[0..29]; removed none
- sheet Relays ports: added OUT[0..23], OUT_HI, OUT_LO, SENSE_HI, SENSE_LO; removed none
- sheet Resisors ports: added OUT_HI, OUT_LO, RSET[0..29], SENSE_HI, SENSE_LO; removed none
Changed lines of the file:
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@@
 (kicad_sch (version 20230121) (generator eeschema)
   (paper "A4")
-  (sheet (at 23.495 87.63) (size 101.6 48.26) (fields_autoplaced)
+  (bus (pts (xy 172.72 90.17) (xy 172.72 96.52))
+    (stroke (width 0) (type default))
+  )
+  (bus (pts (xy 123.19 90.17) (xy 123.19 96.52))
+    (stroke (width 0) (type default))
+  )
+  (wire (pts (xy 142.875 61.595) (xy 146.685 61.595))
+    (stroke (width 0) (type default))
+  )
+  (wire (pts (xy 142.875 64.135) (xy 146.685 64.135))
+    (stroke (width 0) (type default))
+  )
+  (wire (pts (xy 142.875 69.215) (xy 146.685 69.215))
+    (stroke (width 0) (type default))
+  )
+  (wire (pts (xy 142.875 71.755) (xy 146.685 71.755))
+    (stroke (width 0) (type default))
+  )
+  (symbol (lib_id "Mechanical:MountingHole") (at 26.035 177.165 0) (unit 1)
+    (in_bom yes) (on_board yes) (dnp no) (fields_autoplaced)
+    (property "Reference" "H103" (at 29.21 175.895 0)
+      (effects (font (size 1.27 1.27)) (justify left))
+    )
+    (property "Value" "MountingHole" (at 29.21 178.435 0)
+      (effects (font (size 1.27 1.27)) (justify left))
+    )
+    (property "Footprint" "MountingHole:MountingHole_3.2mm_M3_DIN965_Pad_TopBottom" (at 26.035 177.165 0)
+      (effects (font (size 1.27 1.27)) hide)
+    )
+    (property "Datasheet" "~" (at 26.035 177.165 0)
+      (effects (font (size 1.27 1.27)) hide)
+    )
+    (instances
+      (project "ETH1CREF1B"
+        (path "/94724e91-c5c2-46b3-90e6-738f20f45515"
+          (reference "H103") (unit 1)
+        )
+      )
+      (project "ETH1CREF1A"
+        (path "/f534bde3-7724-4aa2-8c73-8f0531e01e95"
+          (reference "H103") (unit 1)
+        )
+      )
+    )
+  )
+  (symbol (lib_id "Mechanical:MountingHole") (at 26.035 170.18 0) (unit 1)
+    (in_bom yes) (on_board yes) (dnp no) (fields_autoplaced)
+    (property "Reference" "H102" (at 29.21 168.91 0)
+      (effects (font (size 1.27 1.27)) (justify left))
+    )
+    (property "Value" "MountingHole" (at 29.21 171.45 0)
+      (effects (font (size 1.27 1.27)) (justify left))
+    )
+    (property "Footprint" "MountingHole:MountingHole_3.2mm_M3_DIN965_Pad_TopBottom" (at 26.035 170.18 0)
+      (effects (font (size 1.27 1.27)) hide)
+    )
+    (property "Datasheet" "~" (at 26.035 170.18 0)
+      (effects (font (size 1.27 1.27)) hide)
+    )
+    (instances
+      (project "ETH1CREF1B"
+        (path "/94724e91-c5c2-46b3-90e6-738f20f45515"
+          (reference "H102") (unit 1)
+        )
+      )
+      (project "ETH1CREF1A"
+        (path "/f534bde3-7724-4aa2-8c73-8f0531e01e95"
+          (reference "H102") (unit 1)
+        )
+      )
+    )
+  )
+  (symbol (lib_id "Mechanical:MountingHole") (at 26.035 163.195 0) (unit 1)
+    (in_bom yes) (on_board yes) (dnp no) (fields_autoplaced)
+    (property "Reference" "H101" (at 29.21 161.925 0)
+      (effects (font (size 1.27 1.27)) (justify left))
+    )
+    (property "Value" "MountingHole" (at 29.21 164.465 0)
+      (effects (font (size 1.27 1.27)) (justify left))
+    )
+    (property "Footprint" "MountingHole:MountingHole_3.2mm_M3_DIN965_Pad_TopBottom" (at 26.035 163.195 0)
+      (effects (font (size 1.27 1.27)) hide)
+    )
+    (property "Datasheet" "~" (at 26.035 163.195 0)
+      (effects (font (size 1.27 1.27)) hide)
+    )
+    (instances
+      (project "ETH1CREF1B"
+        (path "/94724e91-c5c2-46b3-90e6-738f20f45515"
+          (reference "H101") (unit 1)
+        )
+      )
+      (project "ETH1CREF1A"
+        (path "/f534bde3-7724-4aa2-8c73-8f0531e01e95"
+          (reference "H101") (unit 1)
+        )
+      )
+    )
+  )
+  (sheet (at 95.25 96.52) (size 99.06 32.385) (fields_autoplaced)
     (stroke (width 0.1524) (type solid))
     (fill (color 0 0 0 0.0000))
-    (property "Sheetname" "Control" (at 23.495 86.9184 0)
+    (property "Sheetname" "Control" (at 94.5384 128.905 90)
       (effects (font (size 1.27 1.27)) (justify left bottom))
     )
-    (property "Sheetfile" "Control.kicad_sch" (at 23.495 136.4746 0)
+    (property "Sheetfile" "Control.kicad_sch" (at 194.8946 128.905 90)
       (effects (font (size 1.27 1.27)) (justify left top))
+    )
+    (pin "RSET[0..29]" bidirectional (at 123.19 96.52 90)
+      (effects (font (size 1.27 1.27)) (justify right))
+    )
+    (pin "OUT[0..23]" bidirectional (at 172.72 96.52 90)
+      (effects (font (size 1.27 1.27)) (justify right))
     )
     (instances
@@
     )
   )
-  (sheet (at 24.13 21.59) (size 101.6 58.42) (fields_autoplaced)
+  (sheet (at 95.25 58.42) (size 47.625 31.75) (fields_autoplaced)
     (stroke (width 0.1524) (type solid))
     (fill (color 0 0 0 0.0000))
-    (property "Sheetname" "Resisors" (at 24.13 20.8784 0)
+    (property "Sheetname" "Resisors" (at 95.25 57.7084 0)
       (effects (font (size 1.27 1.27)) (justify left bottom))
     )
-    (property "Sheetfile" "Resistors.kicad_sch" (at 24.13 80.5946 0)
+    (property "Sheetfile" "Resistors.kicad_sch" (at 95.25 90.7546 0)
       (effects (font (size 1.27 1.27)) (justify left top))
+    )
+    (pin "RSET[0..29]" bidirectional (at 123.19 90.17 270)
+      (effects (font (size 1.27 1.27)) (justify left))
+    )
+    (pin "OUT_HI" bidirectional (at 142.875 61.595 0)
+      (effects (font (size 1.27 1.27)) (justify right))
+    )
+    (pin "SENSE_HI" bidirectional (at 142.875 64.135 0)
+      (effects (font (size 1.27 1.27)) (justify right))
+    )
+    (pin "SENSE_LO" bidirectional (at 142.875 71.755 0)
+      (effects (font (size 1.27 1.27)) (justify right))
+    )
+    (pin "OUT_LO" bidirectional (at 142.875 69.215 0)
+      (effects (font (size 1.27 1.27)) (justify right))
     )
     (instances
@@
     )
   )
-  (sheet (at 151.765 24.765) (size 90.17 57.15) (fields_autoplaced)
+  (sheet (at 146.685 58.42) (size 47.625 31.75) (fields_autoplaced)
     (stroke (width 0.1524) (type solid))
     (fill (color 0 0 0 0.0000))
-    (property "Sheetname" "Relays" (at 151.765 24.0534 0)
+    (property "Sheetname" "Relays" (at 146.685 57.7084 0)
       (effects (font (size 1.27 1.27)) (justify left bottom))
     )
-    (property "Sheetfile" "Relays.kicad_sch" (at 151.765 82.4996 0)
+    (property "Sheetfile" "Relays.kicad_sch" (at 146.685 90.7546 0)
       (effects (font (size 1.27 1.27)) (justify left top))
     )
+    (pin "OUT_LO" bidirectional (at 146.685 69.215 180)
+      (effects (font (size 1.27 1.27)) (justify left))
+    )
+    (pin "OUT[0..23]" bidirectional (at 172.72 90.17 270)
+      (effects (font (size 1.27 1.27)) (justify left))
+    )
+    (pin "SENSE_LO" bidirectional (at 146.685 71.755 180)
+      (effects (font (size 1.27 1.27)) (justify left))
+    )
+    (pin "OUT_HI" bidirectional (at 146.685 61.595 180)
+      (effects (font (size 1.27 1.27)) (justify left))
+    )
+    (pin "SENSE_HI" bidirectional (at 146.685 64.135 180)
+      (effects (font (size 1.27 1.27)) (justify left))
+    )
     (instances
