File: HARDWARE/ETH1CREF1B/Relays.kicad_sch (KiCad schematic)
At the start: 24 parts, among them J401 Conn_02x06_Odd_Even, K401 9012, K402 9012, K403 9012, K404 9012, K405 9012, K406 9012, K407 9012, K408 9012, K409 9012, K410 9012, K411 9012, K412 9012

Commit message: Hardware
Parts:
- removed D401, D402, D403, D404, D405, D406, D407, D408, D409, D410, D411: 1N4148W, Diode_SMD:D_SOD-123, symbol Diode:1N4148W
- removed K401, K402, K403, K404, K405, K406, K407, K408, K409, K410, K411, K412: 9012, ETH1CREF1A:9012, symbol ETH1CREF1A:9012
- added K401, K402, K403, K404, K405, K406, K407, K408, K409, K410, K411, K412, K413, K414, K415, K416, K417, K418, K419, K420, K421, K422, K423, K424: HE3621A0510, ETH1CREF1B:HE360_x-5050462-8, symbol ETH1CREF1B:HE3621A0510
Connections:
- net +5V: now also K401.2, K402.2, K403.2, K404.2, K405.2, K406.2, K407.2, K408.2, K409.2, K410.2, K411.2, K412.2, K413.2, K414.2, K415.2, K416.2, K417.2, K418.2, K419.2, K420.2, K421.2, K422.2, K423.2, K424.2
- net A: now also K401.4, K407.4, K413.4, K419.4
- net B: now also K402.4, K408.4, K414.4, K420.4
- net C: now also K403.4, K409.4, K415.4, K421.4
- net D: now also K404.4, K410.4, K416.4, K422.4
- net E: now also K405.4, K411.4, K417.4, K423.4
- net F: now also K406.4, K412.4, K418.4, K424.4
- net OUT_HI: now also K401.1, K402.1, K403.1, K404.1, K405.1, K406.1
- net OUT_LO: now also K413.1, K414.1, K415.1, K416.1, K417.1, K418.1
- new net OUT0: K401.3
- new net OUT1: K404.3
- new net OUT10: K408.3
- new net OUT11: K411.3
- new net OUT12: K414.3
- new net OUT13: K417.3
- new net OUT14: K420.3
- new net OUT15: K423.3
- new net OUT16: K403.3
- new net OUT17: K406.3
- new net OUT18: K409.3
- new net OUT19: K412.3
- new net OUT2: K407.3
- new net OUT20: K415.3
- new net OUT21: K418.3
- new net OUT22: K421.3
- new net OUT23: K424.3
- new net OUT3: K410.3
- new net OUT4: K413.3
- new net OUT5: K416.3
- new net OUT6: K419.3
- new net OUT7: K422.3
- new net OUT8: K402.3
- new net OUT9: K405.3
- new net SENSE_HI: K407.1, K408.1, K409.1, K410.1, K411.1, K412.1
- new net SENSE_LO: K419.1, K420.1, K421.1, K422.1, K423.1, K424.1
Other:
- moved on the sheet: J401
